File: pcb/kawaiipad_pcb.kicad_sch (KiCad schematic)
At the start: 28 parts, among them SW1 SW_Push_45deg, SW2 SW_Push_45deg, SW3 SW_Push_45deg, SW4 SW_Push_45deg, SW5 SW_Push_45deg, SW6 SW_Push_45deg, SW7 SW_Push_45deg, SW8 SW_Push_45deg, SW9 SW_Push_45deg, U1 XIAO-RP2040-DIP

Commit message: replace diodes with actual footprint
Parts:
- D1, D2, D3, D4, D5, D6, D7, D8, D9: footprint DiodeLibrary:Diode-Hybrid-Dual -> Diode_THT:D_DO-35_SOD27_P7.62mm_Horizontal
